Commit message: Update file permissions and URDF for Husky Gazebo custom package

File: thesis_custom/urdf/realsense.urdf.xacro (robot description, xacro)
@@ -1,5 +1,5 @@
 <?xml version="1.0"?>
 <robot xmlns:xacro="http://ros.org/wiki/xacro">
-  <link name="front_realsense" />
+  <link name="camera_link" />
   <!--
     The gazebo plugin aligns the depth data with the Z axis, with X=left and Y=up
@@ -7,13 +7,13 @@
     This link only exists to give the gazebo plugin the correctly-oriented frame
   -->
-  <link name="front_realsense_gazebo" />
-  <joint name="front_realsense_gazebo_joint" type="fixed">
-    <parent link="front_realsense"/>
-    <child link="front_realsense_gazebo"/>
+  <link name="camera_link_gazebo" />
+  <joint name="camera_link_gazebo_joint" type="fixed">
+    <parent link="camera_link"/>
+    <child link="camera_link_gazebo"/>
     <origin xyz="0.0 0 0" rpy="-1.5707963267948966 0 -1.5707963267948966"/>
   </joint>
-  <gazebo reference="front_realsense">
+  <gazebo reference="camera_link">
     <turnGravityOff>true</turnGravityOff>
-    <sensor type="depth" name="front_realsense_depth">
+    <sensor type="depth" name="camera_link_depth">
       <update_rate>30</update_rate>
       <camera>
@@ -42,5 +42,5 @@
         <depthImageInfoTopicName>depth/camera_info</depthImageInfoTopicName>
         <pointCloudTopicName>depth/color/points</pointCloudTopicName>
-        <frameName>front_realsense_gazebo</frameName>
+        <frameName>camera_link_gazebo</frameName>
         <pointCloudCutoff>0.105</pointCloudCutoff>
         <pointCloudCutoffMax>8.0</pointCloudCutoffMax>
@@ -59,5 +59,5 @@
   </gazebo>
   <!-- Realsense visual and collision -->
-  <link name="front_realsense_lens">
+  <link name="camera_link_lens">
     <visual>
       <origin xyz="0.02 0 0" rpy="${pi/2} 0 ${pi/2}" />
@@ -74,5 +74,5 @@
     </collision>
   </link>
-  <gazebo reference="front_realsense_lens">
+  <gazebo reference="camera_link_lens">
     <material>Gazebo/Grey</material>
   </gazebo>
@@ -96,14 +96,14 @@
   </link>
   <!-- Joint between the realsense and the aluminum profile -->
-  <joint type="fixed" name="front_realsense_lens_joint">
+  <joint type="fixed" name="camera_link_lens_joint">
     <!-- Offset the camera -->
     <origin xyz="0.005 0 0.45" rpy="0 0 0" />
     <parent link="top_plate_front_link" />
-    <child link="front_realsense_lens" />
+    <child link="camera_link_lens" />
   </joint>
-  <joint type="fixed" name="front_realsense_joint">
+  <joint type="fixed" name="camera_link_joint">
     <origin xyz="0.025 0 0" rpy="0 0 0" />
-    <parent link="front_realsense_lens" />
-    <child link="front_realsense" />
+    <parent link="camera_link_lens" />
+    <child link="camera_link" />
   </joint>
   <!-- Joint between the aluminum profile and the husky -->

Commit message: realsense with correct realsense link name instead of camera_link

File: thesis_custom/urdf/realsense.urdf.xacro (robot description, xacro)
@@ -1,5 +1,5 @@
 <?xml version="1.0"?>
 <robot xmlns:xacro="http://ros.org/wiki/xacro">
-  <link name="camera_link" />
+  <link name="front_realsense" />
   <!--
     The gazebo plugin aligns the depth data with the Z axis, with X=left and Y=up
@@ -7,13 +7,13 @@
     This link only exists to give the gazebo plugin the correctly-oriented frame
   -->
-  <link name="camera_link_gazebo" />
-  <joint name="camera_link_gazebo_joint" type="fixed">
-    <parent link="camera_link"/>
-    <child link="camera_link_gazebo"/>
+  <link name="front_realsense_gazebo" />
+  <joint name="front_realsense_gazebo_joint" type="fixed">
+    <parent link="front_realsense"/>
+    <child link="front_realsense_gazebo"/>
     <origin xyz="0.0 0 0" rpy="-1.5707963267948966 0 -1.5707963267948966"/>
   </joint>
-  <gazebo reference="camera_link">
+  <gazebo reference="front_realsense">
     <turnGravityOff>true</turnGravityOff>
-    <sensor type="depth" name="camera_link_depth">
+    <sensor type="depth" name="front_realsense_depth">
       <update_rate>30</update_rate>
       <camera>
@@ -42,5 +42,5 @@
         <depthImageInfoTopicName>depth/camera_info</depthImageInfoTopicName>
         <pointCloudTopicName>depth/color/points</pointCloudTopicName>
-        <frameName>camera_link_gazebo</frameName>
+        <frameName>front_realsense_gazebo</frameName>
         <pointCloudCutoff>0.105</pointCloudCutoff>
         <pointCloudCutoffMax>8.0</pointCloudCutoffMax>
@@ -59,5 +59,5 @@
   </gazebo>
   <!-- Realsense visual and collision -->
-  <link name="camera_link_lens">
+  <link name="front_realsense_lens">
     <visual>
       <origin xyz="0.02 0 0" rpy="${pi/2} 0 ${pi/2}" />
@@ -74,5 +74,5 @@
     </collision>
   </link>
-  <gazebo reference="camera_link_lens">
+  <gazebo reference="front_realsense_lens">
     <material>Gazebo/Grey</material>
   </gazebo>
@@ -96,14 +96,14 @@
   </link>
   <!-- Joint between the realsense and the aluminum profile -->
-  <joint type="fixed" name="camera_link_lens_joint">
+  <joint type="fixed" name="front_realsense_lens_joint">
     <!-- Offset the camera -->
     <origin xyz="0.005 0 0.45" rpy="0 0 0" />
     <parent link="top_plate_front_link" />
-    <child link="camera_link_lens" />
+    <child link="front_realsense_lens" />
   </joint>
-  <joint type="fixed" name="camera_link_joint">
+  <joint type="fixed" name="front_realsense_joint">
     <origin xyz="0.025 0 0" rpy="0 0 0" />
-    <parent link="camera_link_lens" />
-    <child link="camera_link" />
+    <parent link="front_realsense_lens" />
+    <child link="front_realsense" />
   </joint>
   <!-- Joint between the aluminum profile and the husky -->
